File: kicad/Smiley.kicad_pcb (KiCad board)
At the start: 2 copper layers, 92.4 x 92.4 mm, 28 parts

Commit message: V1.1 01.2024
Parts:
- C1: value 1uF -> 10uF
Changed lines of the file:
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@@
         (effects (font (size 1 1) (thickness 0.15)) (justify mirror))
     )
-    (fp_text value "1uF" (at 1.1 -3.53) (layer "B.SilkS")
+    (fp_text value "10uF" (at 1.1 -3.53) (layer "B.SilkS")
         (effects (font (size 1 1) (thickness 0.15)) (justify mirror))
     )

Commit message: V1.2 02.04.2024
Other:
- board text added: "JLCJLCJLCJLC"

Commit message: V2.0 04.04.2024
Parts:
- moved BAT-HLD-002 34.8 mm to (141.0, 60.0)
- moved G*** 29.0 mm to (164.0, 108.0)
- moved BAT-HLD-002 27.8 mm to (173.5, 60.0)
- moved C1 15.4 mm to (183.0, 88.0)
- moved R1 1.02 mm to (185.5, 66.5), turned to 0 degrees
- moved LP 0.88 mm to (157.0, 49.4)
Routing:
- net Net-(C1-Pad1): track 59.4 -> 108.5 mm
- net Net-(U2-Pad3): track 113.6 -> 78.2 mm
- net Net-(S1-Pad3): track 52.7 -> 87.0 mm
- net Net-(P1-Pad1): track 41.5 -> 30.4 mm
- net Net-(C1-Pad2): track 115.6 -> 123.4 mm
- net Net-(C3-Pad1): track 139.0 -> 133.5 mm, vias 0 -> 1
- net Net-(D7-Pad2): track 92.4 -> 91.6 mm, vias 2 -> 0
- net Net-(D1-Pad2): track 66.8 -> 67.1 mm, vias 3 -> 1
Other:
- board text added: "KHF 04.2024"
- board text removed: "KHF 01.2024"

Commit message: V2 14.04.2024
Parts:
- added ?: , , F.Cu at (146.8, 88.3)
- added Q: LP_rund, !Goody:LP_rund, B.Cu at (170.8, 88.0)
Routing:
- net Net-(U2-Pad3): track 78.2 -> 93.7 mm, vias 0 -> 1
- net Net-(C1-Pad1): track 108.5 -> 95.3 mm
- net Net-(C1-Pad2): track 123.4 -> 133.0 mm
Other:
- board text added: "GND"
Changed lines of the file:
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@@
 		)
 	)
+	(footprint ""
+		(layer "F.Cu")
+		(at 146.8 88.3)
+		(property "Reference" ""
+			(at 0 0 0)
+			(unlocked yes)
+			(layer "F.SilkS")
+			(effects
+				(font
+					(size 1.27 1.27)
+				)
+			)
+		)
+		(property "Value" ""
+			(at 0 0 0)
+			(unlocked yes)
+			(layer "F.Fab")
+			(effects
+				(font
+					(size 1.27 1.27)
+				)
+			)
+		)
+		(property "Footprint" ""
+			(at 0 0 0)
+			(unlocked yes)
+			(layer "F.Fab")
+			(hide yes)
+			(effects
+				(font
+					(size 1.27 1.27)
+				)
+			)
+		)
+		(property "Datasheet" ""
+			(at 0 0 0)
+			(unlocked yes)
+			(layer "F.Fab")
+			(hide yes)
+			(effects
+				(font
+					(size 1.27 1.27)
+				)
+			)
+		)
+		(property "Description" ""
+			(at 0 0 0)
+			(unlocked yes)
+			(layer "F.Fab")
+			(hide yes)
+			(effects
+				(font
+					(size 1.27 1.27)
+				)
+			)
+		)
+		(pad "1" smd circle
+			(at 0 0 180)
+			(size 3 3)
+			(layers "B.Cu" "B.Paste" "B.Mask")
+			(net 2 "Net-(C1-Pad2)")
+		)
+	)
 	(footprint "Capacitor_THT:CP_Radial_D4.0mm_P2.00mm"
 		(layer "B.Cu")
@@
 		(tags "Resistor Axial_DIN0207 series Axial Horizontal pin pitch 7.62mm 0.25W = 1/4W length 6.3mm diameter 2.5mm")
 		(property "Reference" "R1"
-			(at 3.81 2.37 360)
+			(at 3.81 2.37 0)
 			(layer "B.SilkS")
 			(effects
@@
 		)
 		(property "Value" "1,2k"
-			(at 3.81 -2.37 360)
+			(at 3.81 -2.37 0)
 			(layer "B.SilkS")
 			(effects
@@
 		)
 		(fp_text user "${REFERENCE}"
-			(at 3.81 0 360)
+			(at 3.81 0 0)
 			(layer "B.Fab")
 			(effects
@@
 		)
 	)
+	(footprint "!Goody:LP_rund"
+		(layer "B.Cu")
+		(at 170.85 87.95 180)
+		(descr "LP")
+		(property "Reference" "Q"
+			(at -0.15 -3.25 180)
+			(layer "B.SilkS")
+			(effects
+				(font
+					(size 1 1)
+					(thickness 0.15)
+				)
+				(justify mirror)
+			)
+		)
+		(property "Value" "LP_rund"
+			(at 2.54 6 180)
+			(layer "B.Fab")
+			(effects
+				(font
+					(size 1 1)
+					(thickness 0.15)
+				)
+				(justify mirror)
+			)
+		)
+		(property "Footprint" "!Goody:LP_rund"
+			(at 0 0 0)
+			(unlocked yes)
+			(layer "B.Fab")
+			(hide yes)
+			(effects
+				(font
+					(size 1.27 1.27)
+				)
+				(justify mirror)
+			)
+		)
+		(property "Datasheet" ""
+			(at 0 0 0)
+			(unlocked yes)
+			(layer "B.Fab")
+			(hide yes)
+			(effects
+				(font
+					(size 1.27 1.27)
+				)
+				(justify mirror)
+			)
+		)
+		(property "Description" ""
+			(at 0 0 0)
+			(unlocked yes)
+			(layer "B.Fab")
+			(hide yes)
+			(effects
+				(font
+					(size 1.27 1.27)
+				)
+				(justify mirror)
+			)
+		)
+		(attr through_hole)
+		(pad "1" smd circle
+			(at 0 0 180)
+			(size 3 3)
+			(layers "B.Cu" "B.Paste" "B.Mask")
+			(net 16 "Net-(U2-Pad3)")
+		)
+	)
 	(gr_line
 		(start 194.183 86.106)
@@
 	)
 	(gr_text "KHF 04.2024"
-		(at 165 99 0)
+		(at 166 99 0)
 		(layer "B.Cu")
 		(effects
@@
 	)
 	(gr_text "JLCJLCJLCJLC"
-		(at 163 103 0)
+		(at 165 103 0)
 		(layer "B.SilkS")
 		(effects
@@
 	)
 	(gr_text "-"
-		(at 183 67 0)
+		(at 174.9 71.55 0)
 		(layer "B.SilkS")
 		(effects
@@
 		)
 	)
+	(gr_text "GND"
+		(at 148.3 91.8 0)
+		(layer "B.SilkS")
+		(effects
+			(font
+				(size 1 1)
+				(thickness 0.15)
+			)
+			(justify left bottom mirror)
+		)
+	)
 	(gr_text "K"
 		(at 183.2886 104.7091 0)
@@
 	)
 	(gr_text "KHF 04.2024"
-		(at 165 99 0)
+		(at 166 99 0)
 		(layer "B.Mask")
 		(effects
@@
 	)
 	(segment
-		(start 186.44 62.94)
-		(end 190 66.5)
-		(width 0.25)
-		(layer "B.Cu")
-		(net 1)
-	)
-	(segment
-		(start 190 73.2188)
-		(end 191 74.2188)
-		(width 0.25)
-		(layer "B.Cu")
-		(net 1)
-	)
-	(segment
 		(start 190.246 83.693)
 		(end 190.246 78.8797)
@@
 	)
 	(segment
-		(start 190 66.5)
-		(end 190 73.2188)
-		(width 0.25)
-		(layer "B.Cu")
-		(net 1)
-	)
-	(segment
 		(start 167 49.5)
 		(end 166.5 50)
@@
 	)
 	(segment
+		(start 150.15 88.3)
+		(end 153.5086 84.9414)
+		(width 0.25)
+		(layer "B.Cu")
+		(net 2)
+	)
+	(segment
 		(start 154.8486 78.3876)
 		(end 154.8486 82.1391)
@@
 	)
 	(segment
+		(start 153.5086 84.9414)
+		(end 153.5086 83.4791)
+		(width 0.25)
+		(layer "B.Cu")
+		(net 2)
+	)
+	(segment
 		(start 120.9606 72.4611)
 		(end 119.6926 73.7291)
@@
 	)
 	(segment
+		(start 146.8 88.3)
+		(end 150.15 88.3)
+		(width 0.25)
+		(layer "B.Cu")
+		(net 2)
+	)
+	(segment
 		(start 182 71)
 		(end 182 79)
@@
 	)
 	(segment
-		(start 177.2216 74.8741)
-		(end 181.6259 74.8741)
+		(start 181.6259 74.8741)
+		(end 182.2812 74.2188)
 		(width 0.25)
 		(layer "F.Cu")
@@
 	)
 	(segment
-		(start 182.5 74)
-		(end 182.7188 74.2188)
+		(start 177.2216 78.7284)
+		(end 173.9 82.05)
 		(width 0.25)
 		(layer "F.Cu")
@@
 	)
 	(segment
-		(start 182.7188 74.2188)
+		(start 177.2216 74.8741)
+		(end 181.6259 74.8741)
+		(width 0.25)
+		(layer "F.Cu")
+		(net 16)
+	)
+	(segment
+		(start 182.2812 74.2188)
 		(end 185.8137 74.2188)
 		(width 0.25)
@@
 	)
 	(segment
-		(start 181.6259 74.8741)
-		(end 182.5 74)
+		(start 177.2216 74.8741)
+		(end 177.2216 78.7284)
 		(width 0.25)
 		(layer "F.Cu")
 		(net 16)
 	)
+	(via
+		(at 173.9 82.05)
+		(size 0.6)
+		(drill 0.4)
+		(layers "F.Cu" "B.Cu")
+		(net 16)
+	)
 	(segment
 		(start 174.8166 72.4691)
@@
 	)
 	(segment
+		(start 170.85 85.1)
+		(end 170.85 87.95)
+		(width 0.25)
+		(layer "B.Cu")
+		(net 16)
+	)
+	(segment
 		(start 134 68)
 		(end 137 71)
@@
 		(width 0.25)
 		(layer "B.Cu")
+		(net 16)
+	)
+	(segment
+		(start 173.9 82.05)
+		(end 170.85 85.1)
+		(width 0.25)
+		(layer "B.Cu")

Commit message: V 08.05.2024
Other:
- board text added: "KHF 05.2024"
- board text removed: "KHF 04.2024"
Changed lines of the file:
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@@
 			(drillshape 0)
 			(scaleselection 1)
-			(outputdirectory "Smiley_Gerber/")
+			(outputdirectory "SmileyGerber/")
 		)
 	)
@@
 			)
 		)
-		(property "Footprint" ""
+		(property "Footprint" "LED_THT:LED_D5.0mm"
 			(at 0 0 0)
 			(unlocked yes)
@@
 			)
 		)
-		(property "Footprint" ""
+		(property "Footprint" "LED_THT:LED_D5.0mm"
 			(at 0 0 0)
 			(unlocked yes)
@@
 			)
 		)
-		(property "Footprint" ""
+		(property "Footprint" "LED_THT:LED_D5.0mm"
 			(at 0 0 0)
 			(unlocked yes)
@@
 			)
 		)
-		(property "Footprint" ""
+		(property "Footprint" "LED_THT:LED_D5.0mm"
 			(at 0 0 0)
 			(unlocked yes)
@@
 			)
 		)
-		(property "Footprint" ""
+		(property "Footprint" "LED_THT:LED_D5.0mm"
 			(at 0 0 0)
 			(unlocked yes)
@@
 			)
 		)
-		(property "Footprint" ""
+		(property "Footprint" "LED_THT:LED_D5.0mm"
 			(at 0 0 0)
 			(unlocked yes)
@@
 			)
 		)
-		(property "Footprint" ""
+		(property "Footprint" "LED_THT:LED_D5.0mm"
 			(at 0 0 0)
 			(unlocked yes)
@@
 			)
 		)
-		(property "Footprint" ""
+		(property "Footprint" "LED_THT:LED_D5.0mm"
 			(at 0 0 0)
 			(unlocked yes)
@@
 			)
 		)
-		(property "Footprint" ""
+		(property "Footprint" "LED_THT:LED_D5.0mm"
 			(at 0 0 0)
 			(unlocked yes)
@@
 			)
 		)
-		(property "Footprint" ""
+		(property "Footprint" "LED_THT:LED_D5.0mm"
 			(at 0 0 0)
 			(unlocked yes)
@@
 			)
 		)
-		(property "Footprint" ""
+		(property "Footprint" "LED_THT:LED_D5.0mm"
 			(at 0 0 0)
 			(unlocked yes)
@@
 			)
 		)
-		(property "Footprint" ""
+		(property "Footprint" "LED_THT:LED_D5.0mm"
 			(at 0 0 0)
 			(unlocked yes)
@@
 			)
 		)
-		(property "Footprint" ""
+		(property "Footprint" "LED_THT:LED_D5.0mm"
 			(at 0 0 0)
 			(unlocked yes)
@@
 			)
 		)
-		(property "Footprint" ""
+		(property "Footprint" "LED_THT:LED_D5.0mm"
 			(at 0 0 0)
 			(unlocked yes)
@@
 			)
 		)
-		(property "Footprint" ""
+		(property "Footprint" "LED_THT:LED_D5.0mm"
 			(at 0 0 0)
 			(unlocked yes)
@@
 			)
 		)
-		(property "Footprint" ""
+		(property "Footprint" "LOGO"
 			(at 0 0 0)
 			(unlocked yes)
@@
 		(descr "Oberlab-Logo B.SilkS")
 		(property "Reference" "G***"
-			(at -6.445 -11.254 0)
+			(at -7.35 -11.45 0)
 			(layer "B.SilkS")
 			(hide yes)
@@
 		)
 		(property "Value" "LOGO"
-			(at -5.695 -11.254 0)
+			(at -6.6 -11.45 0)
 			(layer "B.SilkS")
 			(hide yes)
@@
 			)
 		)
-		(property "Footprint" ""
+		(property "Footprint" "!Goody:ob-logo_B.SilkS"
 			(at 0 0 0)
 			(unlocked yes)
@@
 			)
 		)
-		(property "Footprint" ""
+		(property "Footprint" "Capacitor_THT:CP_Radial_D4.0mm_P2.00mm"
 			(at 0 0 180)
 			(unlocked yes)
@@
 			)
 		)
-		(property "Footprint" ""
+		(property "Footprint" "Resistor_THT:R_Axial_DIN0207_L6.3mm_D2.5mm_P7.62mm_Horizontal"
 			(at 0 0 0)
 			(unlocked yes)
@@
 			)
 		)
-		(property "Footprint" ""
+		(property "Footprint" "Resistor_THT:R_Axial_DIN0207_L6.3mm_D2.5mm_P7.62mm_Horizontal"
 			(at 0 0 -90)
 			(unlocked yes)
@@
 			)
 		)
-		(property "Footprint" ""
+		(property "Footprint" "Resistor_THT:R_Axial_DIN0207_L6.3mm_D2.5mm_P7.62mm_Horizontal"
 			(at 0 0 90)
 			(unlocked yes)
@@
 			)
 		)
-		(property "Footprint" ""
+		(property "Footprint" "KHF_LIB:Micro_SchalterKHF"
 			(at 0 0 90)
 			(unlocked yes)
@@
 			)
 		)
-		(property "Footprint" ""
+		(property "Footprint" "Package_DIP:DIP-8_W7.62mm"
 			(at 0 0 0)
 			(unlocked yes)
@@
 			)
 		)
-		(property "Footprint" ""
+		(property "Footprint" "Package_DIP:DIP-16_W7.62mm"
 			(at 0 0 180)
 			(unlocked yes)
@@
 		)
 		(property "Value" "Klipp"
-			(at -9.8786 -0.3791 0)
+			(at -8.35 -0.3291 0)
 			(layer "B.SilkS")
 			(effects
@@
 			)
 		)
-		(property "Footprint" ""
+		(property "Footprint" "!Goody:Lötklipp"
 			(at 0 0 0)
 			(unlocked yes)
@@
 			)
 		)
-		(property "Footprint" ""
+		(property "Footprint" "!Goody:Mini-Poti"
 			(at 0 0 180)
 			(unlocked yes)
@@
 		(pad "1" thru_hole circle
 			(at -2.54 -2.54 180)
-			(size 1.524 1.524)
-			(drill 0.762)
+			(size 2 2)
+			(drill 1)
 			(layers "*.Cu" "*.Mask")
 			(remove_unused_layers no)
@@
 		(pad "2" thru_hole circle
 			(at 2.54 -2.54 180)
-			(size 1.524 1.524)
-			(drill 0.762)
+			(size 2 2)
+			(drill 1)
 			(layers "*.Cu" "*.Mask")
 			(remove_unused_layers no)
@@
 		(pad "3" thru_hole circle
 			(at 0 -7.62 180)
-			(size 1.524 1.524)
-			(drill 0.762)
+			(size 2 2)
+			(drill 1)
 			(layers "*.Cu" "*.Mask")
 			(remove_unused_layers no)
@@
 			)
 		)
-		(property "Footprint" ""
+		(property "Footprint" "!Goody:BAT-HLD-SMD-Blech"
 			(at 0 0 0)
 			(unlocked yes)
@@
 			)
 		)
-		(property "Footprint" ""
+		(property "Footprint" "!Goody:BAT-HLD-SMD-Blech"
 			(at 0 0 0)
 			(unlocked yes)
@@
 		(layer "Edge.Cuts")
 	)
-	(gr_text "KHF 04.2024"
-		(at 166 99 0)
+	(gr_text "KHF 05.2024"
+		(at 165.045 98.854 0)
 		(layer "B.Cu")
 		(effects
@@
 	)
 	(gr_text "JLCJLCJLCJLC"
-		(at 165 103 0)
+		(at 167 102.95 0)
 		(layer "B.SilkS")
 		(effects
@@
 		(effects
 			(font
-				(size 1.5 1.5)
-				(thickness 0.3)
+				(size 2 2)
+				(thickness 0.5)
 				(bold yes)
 			)
@@
 		(effects
 			(font
-				(size 1.5 1.5)
-				(thickness 0.3)
+				(size 2 2)
+				(thickness 0.5)
 				(bold yes)
 			)
@@
 		)
 	)
-	(gr_text "KHF 04.2024"
-		(at 166 99 0)
+	(gr_text "KHF 05.2024"
+		(at 165.095 98.804 0)
 		(layer "B.Mask")
 		(effects
