File: kicad-blink/Smiley.kicad_pcb (KiCad board)
At the start: 2 copper layers, 93.3 x 93.4 mm, 31 parts, among them P1 10k, P2 10k, T1 Q_NPN_EBC, T2 Q_NPN_EBC, U1 NE555P, U2 BAT_HLD_SMD

Commit message: V 01.06.24
Connections:
- P1 pad 2: unconnected-(P1-Pad2) -> Net-(D3-A)
- P2 pad 2: unconnected-(P2-Pad2) -> Net-(D3-K)
Routing:
- net Net-(D3-K): track 77.7 -> 84.9 mm
- net Net-(D3-A): track 92.5 -> 96.1 mm
